File: Boards/Main_board/buttonmatrix.kicad_sch (KiCad schematic)
At the start: 43 parts, among them SW1 +, SW10 5, SW11 2, SW12 9, SW13 6, SW14 3, SW15 RSET, SW16 CLR, SW17 PRO, SW18 KEYREL, SW19 ENTR, SW2 -, SW3 0, SW4 VERB, SW5 7, SW6 4, SW7 1, SW8 NOUN, SW9 8

Commit message: First Reroute
Connections:
- net X0: now also SW8.2; no longer SW2.2
- net X1: now also SW2.2; no longer SW8.2
- net X3: now also SW17.2; no longer SW15.2
- net X4: now also SW15.2; no longer SW17.2
- net Y2: no longer D11.1 (K)
- net Y3: now also D11.1 (K)
- net at D2.2 (A): now also SW4.1; no longer SW2.1
- net at D7.2 (A): now also SW6.1; no longer SW7.1
- net at D6.2 (A): now also SW2.1; no longer SW6.1
- net at D8.2 (A): now also SW7.1; no longer SW8.1
- net at SW18.1: now also D19.2 (A); no longer D18.2 (A)
- net at D4.2 (A): now also SW3.1; no longer SW4.1
- net at D3.2 (A): now also SW8.1; no longer SW3.1
- net at SW19.1: now also D17.2 (A); no longer D19.2 (A)
- net at SW17.1: now also D13.2 (A); no longer D17.2 (A)
- net at SW13.1: now also D14.2 (A); no longer D13.2 (A)
- net at SW14.1: now also D15.2 (A); no longer D14.2 (A)
- net at SW15.1: now also D18.2 (A); no longer D15.2 (A)
Other:
- moved on the sheet: D11, SW11, SW13, SW14, SW15, SW17, SW18, SW19, SW2, SW3, SW4, SW6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

Commit message: Completed
Parts:
- renumbered D2 to D1, D14 to D13, D15 to D14, D16 to D15, D13 to D16, D19 to D17, D17 to D18, D18 to D19, D3 to D2, D1 to D3, D6 to D4, D4 to D5, D5 to D6, SW4 to SW1, SW16 to SW15, SW17 to SW16, SW18 to SW17, SW19 to SW18, SW15 to SW19, SW8 to SW2, SW1 to SW3, SW2 to SW4, SW3 to SW5, SW5 to SW6, SW6 to SW7, SW7 to SW8

Commit message: Add main board bom
Parts:
- D1, D10, D11, D12, D13, D14, D15, D16, D17, D18, D19, D2, D3, D4, D5, D6, D7, D8, D9: Link (none) -> https://www.mouser.com/ProductDetail/Vishay-General-Semicon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; Part Number (none) -> S1M-M3/5AT
- R1, R2, R3, R4, R5: Link (none) -> https://www.mouser.com/ProductDetail/652-CR1206FX-1002ELF; Part Number (none) -> CR1206-FX-1002ELF
Changed lines of the file:
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@@
   (title_block
     (title "DSKY Main Board")
-    (date "2024-03-02")
+    (date "2024-03-07")
     (rev "0.3.0")
     (company "Pablo Ortiz López, Evan MacDonald")
@@
       (effects (font (size 1.27 1.27)) hide)
     )
+    (property "Part Number" "S1M-M3/5AT" (at 90.17 54.61 90)
+      (effects (font (size 1.27 1.27)) hide)
+    )
+    (property "Link" "https://www.mouser.com/ProductDetail/Vishay-General-Semiconductor/S1M-M3-5AT?qs=9h5moqLwYqR%2FOw7IjE%252Bumw%3D%3D" (at 90.17 54.61 90)
+      (effects (font (size 1.27 1.27)) hide)
+    )
     (pin "1")
     (pin "2")
@@
       (effects (font (size 1.27 1.27)) hide)
     )
+    (property "Part Number" "S1M-M3/5AT" (at 90.17 54.61 90)
+      (effects (font (size 1.27 1.27)) hide)
+    )
+    (property "Link" "https://www.mouser.com/ProductDetail/Vishay-General-Semiconductor/S1M-M3-5AT?qs=9h5moqLwYqR%2FOw7IjE%252Bumw%3D%3D" (at 90.17 54.61 90)
+      (effects (font (size 1.27 1.27)) hide)
+    )
     (pin "1")
     (pin "2")
@@
       (effects (font (size 1.27 1.27)) hide)
     )
+	(property "Part Number" "CR1206-FX-1002ELF" (at 100.33 35.56 0)
+      (effects (font (size 1.27 1.27)) hide)
+    )
+    (property "Link" "https://www.mouser.com/ProductDetail/652-CR1206FX-1002ELF" (at 100.33 35.56 0)
+      (effects (font (size 1.27 1.27)) hide)
+    )
     (pin "1")
     (pin "2")
@@
       (effects (font (size 1.27 1.27)) hide)
     )
+    (property "Part Number" "S1M-M3/5AT" (at 90.17 54.61 90)
+      (effects (font (size 1.27 1.27)) hide)
+    )
+    (property "Link" "https://www.mouser.com/ProductDetail/Vishay-General-Semiconductor/S1M-M3-5AT?qs=9h5moqLwYqR%2FOw7IjE%252Bumw%3D%3D" (at 90.17 54.61 90)
+      (effects (font (size 1.27 1.27)) hide)
+    )
     (pin "1")
     (pin "2")
@@
       (effects (font (size 1.27 1.27)) hide)
     )
+    (property "Part Number" "S1M-M3/5AT" (at 90.17 54.61 90)
+      (effects (font (size 1.27 1.27)) hide)
+    )
+    (property "Link" "https://www.mouser.com/ProductDetail/Vishay-General-Semiconductor/S1M-M3-5AT?qs=9h5moqLwYqR%2FOw7IjE%252Bumw%3D%3D" (at 90.17 54.61 90)
+      (effects (font (size 1.27 1.27)) hide)
+    )
     (pin "1")
     (pin "2")
@@
       (effects (font (size 1.27 1.27)) hide)
     )
+    (property "Part Number" "S1M-M3/5AT" (at 90.17 54.61 90)
+      (effects (font (size 1.27 1.27)) hide)
+    )
+    (property "Link" "https://www.mouser.com/ProductDetail/Vishay-General-Semiconductor/S1M-M3-5AT?qs=9h5moqLwYqR%2FOw7IjE%252Bumw%3D%3D" (at 90.17 54.61 90)
+      (effects (font (size 1.27 1.27)) hide)
+    )
     (pin "1")
     (pin "2")
@@
       (effects (font (size 1.27 1.27)) hide)
     )
+    (property "Part Number" "S1M-M3/5AT" (at 90.17 54.61 90)
+      (effects (font (size 1.27 1.27)) hide)
+    )
+    (property "Link" "https://www.mouser.com/ProductDetail/Vishay-General-Semiconductor/S1M-M3-5AT?qs=9h5moqLwYqR%2FOw7IjE%252Bumw%3D%3D" (at 90.17 54.61 90)
+      (effects (font (size 1.27 1.27)) hide)
+    )
     (pin "1")
     (pin "2")
@@
       (effects (font (size 1.27 1.27)) hide)
     )
+    (property "Part Number" "CR1206-FX-1002ELF" (at 100.33 35.56 0)
+      (effects (font (size 1.27 1.27)) hide)
+    )
+    (property "Link" "https://www.mouser.com/ProductDetail/652-CR1206FX-1002ELF" (at 100.33 35.56 0)
+      (effects (font (size 1.27 1.27)) hide)
+    )
     (pin "1")
     (pin "2")
@@
       (effects (font (size 1.27 1.27)) hide)
     )
+	(property "Part Number" "CR1206-FX-1002ELF" (at 100.33 35.56 0)
+      (effects (font (size 1.27 1.27)) hide)
+    )
+    (property "Link" "https://www.mouser.com/ProductDetail/652-CR1206FX-1002ELF" (at 100.33 35.56 0)
+      (effects (font (size 1.27 1.27)) hide)
+    )
     (pin "1")
     (pin "2")
@@
       (effects (font (size 1.27 1.27)) hide)
     )
+    (property "Part Number" "S1M-M3/5AT" (at 90.17 54.61 90)
+      (effects (font (size 1.27 1.27)) hide)
+    )
+    (property "Link" "https://www.mouser.com/ProductDetail/Vishay-General-Semiconductor/S1M-M3-5AT?qs=9h5moqLwYqR%2FOw7IjE%252Bumw%3D%3D" (at 90.17 54.61 90)
+      (effects (font (size 1.27 1.27)) hide)
+    )
     (pin "1")
     (pin "2")
@@
       (effects (font (size 1.27 1.27)) hide)
     )
+	(property "Part Number" "CR1206-FX-1002ELF" (at 100.33 35.56 0)
+      (effects (font (size 1.27 1.27)) hide)
+    )
+    (property "Link" "https://www.mouser.com/ProductDetail/652-CR1206FX-1002ELF" (at 100.33 35.56 0)
+      (effects (font (size 1.27 1.27)) hide)
+    )
     (pin "1")
     (pin "2")
@@
       (effects (font (size 1.27 1.27)) hide)
     )
+    (property "Part Number" "S1M-M3/5AT" (at 90.17 54.61 90)
+      (effects (font (size 1.27 1.27)) hide)
+    )
+    (property "Link" "https://www.mouser.com/ProductDetail/Vishay-General-Semiconductor/S1M-M3-5AT?qs=9h5moqLwYqR%2FOw7IjE%252Bumw%3D%3D" (at 90.17 54.61 90)
+      (effects (font (size 1.27 1.27)) hide)
+    )
     (pin "1")
     (pin "2")
@@
       (effects (font (size 1.27 1.27)) hide)
     )
+    (property "Part Number" "S1M-M3/5AT" (at 90.17 54.61 90)
+      (effects (font (size 1.27 1.27)) hide)
+    )
+    (property "Link" "https://www.mouser.com/ProductDetail/Vishay-General-Semiconductor/S1M-M3-5AT?qs=9h5moqLwYqR%2FOw7IjE%252Bumw%3D%3D" (at 90.17 54.61 90)
+      (effects (font (size 1.27 1.27)) hide)
+    )
     (pin "1")
     (pin "2")
@@
       (effects (font (size 1.27 1.27)) hide)
     )
+	(property "Part Number" "CR1206-FX-1002ELF" (at 100.33 35.56 0)
+      (effects (font (size 1.27 1.27)) hide)
+    )
+    (property "Link" "https://www.mouser.com/ProductDetail/652-CR1206FX-1002ELF" (at 100.33 35.56 0)
+      (effects (font (size 1.27 1.27)) hide)
+    )
     (pin "1")
     (pin "2")
@@
       (effects (font (size 1.27 1.27)) hide)
     )
+    (property "Part Number" "S1M-M3/5AT" (at 90.17 54.61 90)
+      (effects (font (size 1.27 1.27)) hide)
+    )
+    (property "Link" "https://www.mouser.com/ProductDetail/Vishay-General-Semiconductor/S1M-M3-5AT?qs=9h5moqLwYqR%2FOw7IjE%252Bumw%3D%3D" (at 90.17 54.61 90)
+      (effects (font (size 1.27 1.27)) hide)
+    )
     (pin "1")
     (pin "2")
@@
       (effects (font (size 1.27 1.27)) hide)
     )
+    (property "Part Number" "S1M-M3/5AT" (at 90.17 54.61 90)
+      (effects (font (size 1.27 1.27)) hide)
+    )
+    (property "Link" "https://www.mouser.com/ProductDetail/Vishay-General-Semiconductor/S1M-M3-5AT?qs=9h5moqLwYqR%2FOw7IjE%252Bumw%3D%3D" (at 90.17 54.61 90)
+      (effects (font (size 1.27 1.27)) hide)
+    )
     (pin "1")
     (pin "2")
@@
       (effects (font (size 1.27 1.27)) hide)
     )
+    (property "Part Number" "S1M-M3/5AT" (at 90.17 54.61 90)
+      (effects (font (size 1.27 1.27)) hide)
+    )
+    (property "Link" "https://www.mouser.com/ProductDetail/Vishay-General-Semiconductor/S1M-M3-5AT?qs=9h5moqLwYqR%2FOw7IjE%252Bumw%3D%3D" (at 90.17 54.61 90)
+      (effects (font (size 1.27 1.27)) hide)
+    )
     (pin "1")
     (pin "2")
@@
       (effects (font (size 1.27 1.27)) hide)
     )
+    (property "Part Number" "S1M-M3/5AT" (at 90.17 54.61 90)
+      (effects (font (size 1.27 1.27)) hide)
+    )
+    (property "Link" "https://www.mouser.com/ProductDetail/Vishay-General-Semiconductor/S1M-M3-5AT?qs=9h5moqLwYqR%2FOw7IjE%252Bumw%3D%3D" (at 90.17 54.61 90)
+      (effects (font (size 1.27 1.27)) hide)
+    )
     (pin "1")
     (pin "2")
@@
       (effects (font (size 1.27 1.27)) hide)
     )
+    (property "Part Number" "S1M-M3/5AT" (at 90.17 54.61 90)
+      (effects (font (size 1.27 1.27)) hide)
+    )
+    (property "Link" "https://www.mouser.com/ProductDetail/Vishay-General-Semiconductor/S1M-M3-5AT?qs=9h5moqLwYqR%2FOw7IjE%252Bumw%3D%3D" (at 90.17 54.61 90)
+      (effects (font (size 1.27 1.27)) hide)
+    )
     (pin "1")
     (pin "2")
@@
       (effects (font (size 1.27 1.27)) hide)
     )
+    (property "Part Number" "S1M-M3/5AT" (at 90.17 54.61 90)
+      (effects (font (size 1.27 1.27)) hide)
+    )
+    (property "Link" "https://www.mouser.com/ProductDetail/Vishay-General-Semiconductor/S1M-M3-5AT?qs=9h5moqLwYqR%2FOw7IjE%252Bumw%3D%3D" (at 90.17 54.61 90)
+      (effects (font (size 1.27 1.27)) hide)
+    )
     (pin "1")
     (pin "2")
@@
       (effects (font (size 1.27 1.27)) hide)
     )
+    (property "Part Number" "S1M-M3/5AT" (at 90.17 54.61 90)
+      (effects (font (size 1.27 1.27)) hide)
+    )
+    (property "Link" "https://www.mouser.com/ProductDetail/Vishay-General-Semiconductor/S1M-M3-5AT?qs=9h5moqLwYqR%2FOw7IjE%252Bumw%3D%3D" (at 90.17 54.61 90)
+      (effects (font (size 1.27 1.27)) hide)
+    )
     (pin "1")
     (pin "2")
@@
       (effects (font (size 1.27 1.27)) hide)
     )
+    (property "Part Number" "S1M-M3/5AT" (at 90.17 54.61 90)
+      (effects (font (size 1.27 1.27)) hide)
+    )
+    (property "Link" "https://www.mouser.com/ProductDetail/Vishay-General-Semiconductor/S1M-M3-5AT?qs=9h5moqLwYqR%2FOw7IjE%252Bumw%3D%3D" (at 90.17 54.61 90)
+      (effects (font (size 1.27 1.27)) hide)
+    )
     (pin "1")
     (pin "2")
@@
       (effects (font (size 1.27 1.27)) hide)
     )
+    (property "Part Number" "S1M-M3/5AT" (at 90.17 54.61 90)
+      (effects (font (size 1.27 1.27)) hide)
+    )
+    (property "Link" "https://www.mouser.com/ProductDetail/Vishay-General-Semiconductor/S1M-M3-5AT?qs=9h5moqLwYqR%2FOw7IjE%252Bumw%3D%3D" (at 90.17 54.61 90)
+      (effects (font (size 1.27 1.27)) hide)
+    )
     (pin "1")
     (pin "2")
@@
       (effects (font (size 1.27 1.27)) hide)
     )
+    (property "Part Number" "S1M-M3/5AT" (at 90.17 54.61 90)
+      (effects (font (size 1.27 1.27)) hide)
+    )
+    (property "Link" "https://www.mouser.com/ProductDetail/Vishay-General-Semiconductor/S1M-M3-5AT?qs=9h5moqLwYqR%2FOw7IjE%252Bumw%3D%3D" (at 90.17 54.61 90)
+      (effects (font (size 1.27 1.27)) hide)
+    )
