File: Boards/Main_board/backlight.kicad_sch (KiCad schematic)
At the start: 43 parts, among them Q2 SI2306

Commit message: Routing of mainboard with backlight
Parts:
- R10, R11, R12, R13, R14, R15, R16, R17, R18, R19, R20, R21, R22, R23, R24, R25, R26, R27, R9: footprint (none) -> Resistor_SMD:R_1206_3216Metric
- R6, R7, R8: footprint Resistor_SMD:R_1206_3216Metric_Pad1.30x1.75mm_HandSolder -> Resistor_SMD:R_1206_3216Metric
Changed lines of the file:
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@@
 			)
 		)
-		(property "Footprint" "Resistor_SMD:R_1206_3216Metric_Pad1.30x1.75mm_HandSolder"
+		(property "Footprint" "Resistor_SMD:R_1206_3216Metric"
 			(at 232.41 73.66 0)
 			(effects
@@
 			)
 		)
-		(property "Footprint" ""
+		(property "Footprint" "Resistor_SMD:R_1206_3216Metric"
 			(at 33.02 68.58 0)
 			(effects
@@
 			)
 		)
-		(property "Footprint" ""
+		(property "Footprint" "Resistor_SMD:R_1206_3216Metric"
 			(at 104.14 68.58 0)
 			(effects
@@
 			)
 		)
-		(property "Footprint" ""
+		(property "Footprint" "Resistor_SMD:R_1206_3216Metric"
 			(at 166.37 68.58 0)
 			(effects
@@
 			)
 		)
-		(property "Footprint" ""
+		(property "Footprint" "Resistor_SMD:R_1206_3216Metric"
 			(at 68.58 68.58 0)
 			(effects
@@
 			)
 		)
-		(property "Footprint" ""
+		(property "Footprint" "Resistor_SMD:R_1206_3216Metric"
 			(at 121.92 68.58 0)
 			(effects
@@
 			)
 		)
-		(property "Footprint" ""
+		(property "Footprint" "Resistor_SMD:R_1206_3216Metric"
 			(at 59.69 68.58 0)
 			(effects
@@
 			)
 		)
-		(property "Footprint" ""
+		(property "Footprint" "Resistor_SMD:R_1206_3216Metric"
 			(at 148.59 68.58 0)
 			(effects
@@
 			)
 		)
-		(property "Footprint" ""
+		(property "Footprint" "Resistor_SMD:R_1206_3216Metric"
 			(at 184.15 68.58 0)
 			(effects
@@
 			)
 		)
-		(property "Footprint" ""
+		(property "Footprint" "Resistor_SMD:R_1206_3216Metric"
 			(at 41.91 68.58 0)
 			(effects
@@
 			)
 		)
-		(property "Footprint" ""
+		(property "Footprint" "Resistor_SMD:R_1206_3216Metric"
 			(at 139.7 68.58 0)
 			(effects
@@
 			)
 		)
-		(property "Footprint" ""
+		(property "Footprint" "Resistor_SMD:R_1206_3216Metric"
 			(at 157.48 68.58 0)
 			(effects
@@
 			)
 		)
-		(property "Footprint" "Resistor_SMD:R_1206_3216Metric_Pad1.30x1.75mm_HandSolder"
+		(property "Footprint" "Resistor_SMD:R_1206_3216Metric"
 			(at 233.68 121.92 0)
 			(effects
@@
 			)
 		)
-		(property "Footprint" ""
+		(property "Footprint" "Resistor_SMD:R_1206_3216Metric"
 			(at 130.81 68.58 0)
 			(effects
@@
 			)
 		)
-		(property "Footprint" "Resistor_SMD:R_1206_3216Metric_Pad1.30x1.75mm_HandSolder"
+		(property "Footprint" "Resistor_SMD:R_1206_3216Metric"
 			(at 227.33 78.74 0)
 			(effects
@@
 			)
 		)
-		(property "Footprint" ""
+		(property "Footprint" "Resistor_SMD:R_1206_3216Metric"
 			(at 86.36 68.58 0)
 			(effects
@@
 			)
 		)
-		(property "Footprint" ""
+		(property "Footprint" "Resistor_SMD:R_1206_3216Metric"
 			(at 95.25 68.58 0)
 			(effects
@@
 			)
 		)
-		(property "Footprint" ""
+		(property "Footprint" "Resistor_SMD:R_1206_3216Metric"
 			(at 113.03 68.58 0)
 			(effects
@@
 			)
 		)
-		(property "Footprint" ""
+		(property "Footprint" "Resistor_SMD:R_1206_3216Metric"
 			(at 24.13 68.58 0)
 			(effects
@@
 			)
 		)
-		(property "Footprint" ""
+		(property "Footprint" "Resistor_SMD:R_1206_3216Metric"
 			(at 50.8 68.58 0)
 			(effects
@@
 			)
 		)
-		(property "Footprint" ""
+		(property "Footprint" "Resistor_SMD:R_1206_3216Metric"
 			(at 175.26 68.58 0)
 			(effects
@@
 			)
 		)
-		(property "Footprint" ""
+		(property "Footprint" "Resistor_SMD:R_1206_3216Metric"
 			(at 77.47 68.58 0)
 			(effects

Commit message: Remove dummy load and fix silkscreen collisions
Parts:
- removed R8: 1k, Resistor_SMD:R_1206_3216Metric, symbol Device:R_Small
- D1, D10, D11, D12, D13, D14, D15, D16, D17, D18, D19, D2, D3, D4, D5, D6, D7, D8, D9: footprint Libraries:MX-LED-PolarityMarked -> Switch_Misc:MX-LED-PolarityMarked
Other:
- note added: "LS PWM Switch"
- note removed: "LS PWM Switch w/ 1k dummy resistive load"
Changed lines of the file:
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@@
 	)
 	(junction
-		(at 250.19 121.92)
-		(diameter 0)
-		(color 0 0 0 0)
-	)
-	(junction
 		(at 175.26 95.25)
 		(diameter 0)
@@
 	(wire
 		(pts
-			(xy 231.14 132.08) (xy 242.57 132.08)
+			(xy 237.49 132.08) (xy 242.57 132.08)
 		)
 		(stroke
@@
 	(wire
 		(pts
-			(xy 250.19 121.92) (xy 250.19 127)
-		)
-		(stroke
-			(width 0)
-			(type default)
-		)
-	)
-	(wire
-		(pts
-			(xy 250.19 113.03) (xy 250.19 121.92)
+			(xy 250.19 113.03) (xy 250.19 127)
 		)
 		(stroke
@@
 	(wire
 		(pts
-			(xy 222.25 116.84) (xy 222.25 121.92)
-		)
-		(stroke
-			(width 0)
-			(type default)
-		)
-	)
-	(wire
-		(pts
 			(xy 113.03 95.25) (xy 104.14 95.25)
 		)
@@
 	(wire
 		(pts
-			(xy 236.22 121.92) (xy 250.19 121.92)
-		)
-		(stroke
-			(width 0)
-			(type default)
-		)
-	)
-	(wire
-		(pts
 			(xy 139.7 80.01) (xy 139.7 95.25)
 		)
@@
 	(wire
 		(pts
-			(xy 222.25 121.92) (xy 231.14 121.92)
-		)
-		(stroke
-			(width 0)
-			(type default)
-		)
-	)
-	(wire
-		(pts
 			(xy 175.26 66.04) (xy 175.26 62.23)
 		)
@@
 		)
 	)
-	(text "LS PWM Switch w/ 1k dummy resistive load"
+	(text "LS PWM Switch"
 		(exclude_from_sim no)
-		(at 215.9 109.22 0)
+		(at 235.712 109.728 0)
 		(effects
 			(font
@@
 	(global_label "PWMfilt"
 		(shape input)
-		(at 231.14 132.08 180)
+		(at 237.49 132.08 180)
 		(fields_autoplaced yes)
 		(effects
@@
 		)
 		(property "Intersheetrefs" "${INTERSHEET_REFS}"
-			(at 221.2606 132.08 0)
+			(at 227.6106 132.08 0)
 			(effects
 				(font
@@
 			)
 		)
-		(property "Footprint" "Libraries:MX-LED-PolarityMarked"
+		(property "Footprint" "Switch_Misc:MX-LED-PolarityMarked"
 			(at 157.48 77.47 90)
 			(effects
@@
 			)
 		)
-		(property "Footprint" "Libraries:MX-LED-PolarityMarked"
+		(property "Footprint" "Switch_Misc:MX-LED-PolarityMarked"
 			(at 68.58 77.47 90)
 			(effects
@@
 			)
 		)
-		(property "Footprint" "Libraries:MX-LED-PolarityMarked"
+		(property "Footprint" "Switch_Misc:MX-LED-PolarityMarked"
 			(at 148.59 77.47 90)
 			(effects
@@
 			)
 		)
-		(property "Footprint" "Libraries:MX-LED-PolarityMarked"
+		(property "Footprint" "Switch_Misc:MX-LED-PolarityMarked"
 			(at 50.8 77.47 90)
 			(effects
@@
 			)
 		)
-		(property "Footprint" "Libraries:MX-LED-PolarityMarked"
+		(property "Footprint" "Switch_Misc:MX-LED-PolarityMarked"
 			(at 77.47 77.47 90)
 			(effects
@@
 			)
 		)
-		(property "Footprint" "Libraries:MX-LED-PolarityMarked"
+		(property "Footprint" "Switch_Misc:MX-LED-PolarityMarked"
 			(at 33.02 77.47 90)
 			(effects
@@
 			)
 		)
-		(property "Footprint" "Libraries:MX-LED-PolarityMarked"
+		(property "Footprint" "Switch_Misc:MX-LED-PolarityMarked"
 			(at 139.7 77.47 90)
 			(effects
@@
 			)
 		)
-		(property "Footprint" "Libraries:MX-LED-PolarityMarked"
+		(property "Footprint" "Switch_Misc:MX-LED-PolarityMarked"
 			(at 130.81 77.47 90)
 			(effects
@@
 			)
 		)
-		(property "Footprint" "Libraries:MX-LED-PolarityMarked"
+		(property "Footprint" "Switch_Misc:MX-LED-PolarityMarked"
 			(at 59.69 77.47 90)
 			(effects
@@
 			)
 		)
-		(property "Footprint" "Libraries:MX-LED-PolarityMarked"
+		(property "Footprint" "Switch_Misc:MX-LED-PolarityMarked"
 			(at 95.25 77.47 90)
 			(effects
@@
 	(symbol
 		(lib_id "Device:R_Small")
-		(at 233.68 121.92 270)
-		(unit 1)
-		(exclude_from_sim no)
-		(in_bom yes)
-		(on_board yes)
-		(dnp no)
-		(fields_autoplaced yes)
-		(property "Reference" "R8"
-			(at 233.68 116.84 90)
-			(effects
-				(font
-					(size 1.27 1.27)
-				)
-			)
-		)
-		(property "Value" "1k"
-			(at 233.68 119.38 90)
-			(effects
-				(font
-					(size 1.27 1.27)
-				)
-			)
-		)
-		(property "Footprint" "Resistor_SMD:R_1206_3216Metric"
-			(at 233.68 121.92 0)
-			(effects
-				(font
-					(size 1.27 1.27)
-				)
-				(hide yes)
-			)
-		)
-		(property "Datasheet" "~"
-			(at 233.68 121.92 0)
-			(effects
-				(font
-					(size 1.27 1.27)
-				)
-				(hide yes)
-			)
-		)
-		(property "Description" ""
-			(at 233.68 121.92 0)
-			(effects
-				(font
-					(size 1.27 1.27)
-				)
-				(hide yes)
-			)
-		)
-		(property "Part Number" "CR1206-FX-1001ELF"
-			(at 285.75 121.92 90)
-			(effects
-				(font
-					(size 1.27 1.27)
-				)
-				(hide yes)
-			)
-		)
-		(property "Link" "https://www.mouser.com/ProductDetail/652-CR1206FX-1001ELF"
-			(at 285.75 121.92 90)
-			(effects
-				(font
-					(size 1.27 1.27)
-				)
-				(hide yes)
-			)
-		)
-		(pin "1"
-		)
-		(pin "2"
-		)
-		(instances
-			(project "Main_board"
-				(path "/f30854c1-5bc2-470d-aabe-1768a5b01b46/6de8313f-adfc-4236-b602-98157f8335d8"
-					(reference "R8")
-					(unit 1)
-				)
-			)
-		)
-	)
-	(symbol
-		(lib_id "Device:R_Small")
 		(at 130.81 68.58 0)
 		(unit 1)
@@
 			)
 		)
-		(property "Footprint" "Libraries:MX-LED-PolarityMarked"
+		(property "Footprint" "Switch_Misc:MX-LED-PolarityMarked"
 			(at 184.15 77.47 90)
 			(effects
@@
 			)
 		)
-		(property "Footprint" "Libraries:MX-LED-PolarityMarked"
+		(property "Footprint" "Switch_Misc:MX-LED-PolarityMarked"
 			(at 175.26 77.47 90)
 			(effects
@@
 	)
 	(symbol
-		(lib_id "power:+5V")
-		(at 222.25 116.84 0)
-		(unit 1)
-		(exclude_from_sim no)
-		(in_bom yes)
-		(on_board yes)
-		(dnp no)
-		(fields_autoplaced yes)
-		(property "Reference" "#PWR018"
-			(at 222.25 120.65 0)
-			(effects
-				(font
-					(size 1.27 1.27)
-				)
-				(hide yes)
-			)
-		)
-		(property "Value" "+5V"
-			(at 222.25 111.76 0)
-			(effects
-				(font
-					(size 1.27 1.27)
-				)
-			)
-		)
-		(property "Footprint" ""
-			(at 222.25 116.84 0)
-			(effects
-				(font
-					(size 1.27 1.27)
-				)
-				(hide yes)
-			)
-		)
-		(property "Datasheet" ""
-			(at 222.25 116.84 0)
-			(effects
-				(font
-					(size 1.27 1.27)
-				)
-				(hide yes)
-			)
-		)
-		(property "Description" ""
-			(at 222.25 116.84 0)
-			(effects
-				(font
-					(size 1.27 1.27)
-				)
-				(hide yes)
-			)
-		)
-		(pin "1"
-		)
-		(instances
-			(project "Main_board"
-				(path "/f30854c1-5bc2-470d-aabe-1768a5b01b46/6de8313f-adfc-4236-b602-98157f8335d8"
-					(reference "#PWR018")
-					(unit 1)
-				)
-			)
-		)
-	)
-	(symbol
 		(lib_id "Device:R_Small")
 		(at 113.03 68.58 0)
@@
 			)
 		)
-		(property "Footprint" "Libraries:MX-LED-PolarityMarked"
+		(property "Footprint" "Switch_Misc:MX-LED-PolarityMarked"
 			(at 113.03 77.47 90)
 			(effects
@@
 			)
 		)
-		(property "Footprint" "Libraries:MX-LED-PolarityMarked"
+		(property "Footprint" "Switch_Misc:MX-LED-PolarityMarked"
 			(at 24.13 77.47 90)
 			(effects
@@
 			)
 		)
-		(property "Footprint" "Libraries:MX-LED-PolarityMarked"
+		(property "Footprint" "Switch_Misc:MX-LED-PolarityMarked"
 			(at 121.92 77.47 90)
 			(effects
@@
 			)
 		)
-		(property "Footprint" "Libraries:MX-LED-PolarityMarked"
+		(property "Footprint" "Switch_Misc:MX-LED-PolarityMarked"
 			(at 166.37 77.47 90)
 			(effects
@@
 			)
 		)
-		(property "Footprint" "Libraries:MX-LED-PolarityMarked"
+		(property "Footprint" "Switch_Misc:MX-LED-PolarityMarked"
 			(at 104.14 77.47 90)
 			(effects
@@
 			)
 		)
-		(property "Footprint" "Libraries:MX-LED-PolarityMarked"
+		(property "Footprint" "Switch_Misc:MX-LED-PolarityMarked"
 			(at 86.36 77.47 90)
 			(effects
@@
 			)
 		)
-		(property "Footprint" "Libraries:MX-LED-PolarityMarked"
+		(property "Footprint" "Switch_Misc:MX-LED-PolarityMarked"
 			(at 41.91 77.47 90)
 			(effects
