File: Boards/Single_board/Single_board.kicad_sch (KiCad schematic)
At the start: 8 parts, among them J1 Conn_01x04_Socket, J2 Conn_01x04_Socket, Q1 SI2306

Commit message: some progress on the arduino boilerplate
Parts:
- removed A1: Arduino_Nano_Socket, PCM_arduino-library:Arduino_Nano_Socket, symbol PCM_arduino-library:Arduino_Nano_Socket
- C1: footprint Capacitor_SMD:C_1206_3216Metric_Pad1.33x1.80mm_HandSolder -> Capacitor_SMD:C_0805_2012Metric
- Q1: footprint Package_TO_SOT_SMD:SOT-23-3 -> Package_TO_SOT_SMD:SOT-23
- R1, R2, R3: footprint Resistor_SMD:R_1206_3216Metric_Pad1.30x1.75mm_HandSolder -> Resistor_SMD:R_1206_3216Metric
Connections:
- no-connect marks 10 -> 0
Other:
- added sheet Atmega 328P (328p.kicad_sch)
- added sheet USB-C (usb.kicad_sch)
- title: DSKY Main Board -> DSKY Board
- moved on the sheet: J1, J2

Commit message: Single board nearly ready to order
Parts:
- added J4: ICSP, Connector_PinHeader_2.54mm:PinHeader_2x03_P2.54mm_Vertical_SMD, symbol Connector:Conn_01x06_Pin
- added R48: 0, Jumper:SolderJumper-2_P1.3mm_Open_RoundedPad1.0x1.5mm, symbol Device:R_Small
- J1: value Conn_01x04_Socket -> AUX_I2C_1
- J2: value Conn_01x04_Socket -> AUX_I2C_2
Connections:
- net +5V: now also J4.2 (Pin_2)
- net GND: now also J4.6 (Pin_6)
- net PWMcom: now also R48.1; no longer Q1.3 (D), R2.1
- new net: Q1.3 (D), R2.1, R48.2
- new net MISO: J4.1 (Pin_1)
- new net MOSI: J4.4 (Pin_4)
- new net RESET: J4.5 (Pin_5)
- new net SCK: J4.3 (Pin_3)
Other:
- sheet Atmega 328P ports: added 5V, CS, GND, MISO, MOSI, PWM, RESET, SCK, SCL, SDA, UC_RX, UC_TX, X0, X1, X2, X3, X4, Y0, Y1, Y2, Y3; removed none
- sheet USB-C ports: added 5V, GND, RESET, USB_RX, USB_TX; removed none
- moved on the sheet: J1, J2

Commit message: Fixes on single board
Other:
- sheet Alarm_lights ports: added 5V, GND, SCL, SDA; removed none

Commit message: Visual Schematic improvements
Connections:
- net PWMcom renamed PWMCom
Other:
- sheet Alarm_lights renamed Alarm Lights
- sheet Alarm Lights ports: added PWMCom; removed none
- sheet Keyboard Backlight ports: added PWMCom; removed GND, PWM
Changed lines of the file:
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@@
 	(wire
 		(pts
+			(xy 236.22 125.73) (xy 240.03 125.73)
+		)
+		(stroke
+			(width 0)
+			(type default)
+		)
+	)
+	(wire
+		(pts
 			(xy 64.77 45.72) (xy 81.28 45.72)
 		)
@@
 	(wire
 		(pts
-			(xy 67.31 67.31) (xy 71.12 67.31)
+			(xy 67.31 74.93) (xy 71.12 74.93)
 		)
 		(stroke
@@
 		)
 	)
+	(wire
+		(pts
+			(xy 38.1 74.93) (xy 43.18 74.93)
+		)
+		(stroke
+			(width 0)
+			(type default)
+		)
+	)
 	(bus
 		(pts
@@
 		)
 	)
-	(wire
-		(pts
-			(xy 67.31 72.39) (xy 72.39 72.39)
-		)
-		(stroke
-			(width 0)
-			(type default)
-		)
-	)
 	(bus
 		(pts
@@
 		)
 	)
-	(wire
-		(pts
-			(xy 39.37 74.93) (xy 43.18 74.93)
-		)
-		(stroke
-			(width 0)
-			(type default)
-		)
-	)
 	(rectangle
 		(start 222.25 98.425)
@@
 		)
 	)
+	(global_label "PWMCom"
+		(shape input)
+		(at 38.1 74.93 180)
+		(fields_autoplaced yes)
+		(effects
+			(font
+				(size 1.27 1.27)
+			)
+			(justify right)
+		)
+		(property "Intersheetrefs" "${INTERSHEET_REFS}"
+			(at 26.8297 74.93 0)
+			(effects
+				(font
+					(size 1.27 1.27)
+				)
+				(justify right)
+				(hide yes)
+			)
+		)
+	)
 	(global_label "RESET"
 		(shape input)
@@
 		)
 	)
-	(global_label "PWMcom"
+	(global_label "PWMCom"
 		(shape input)
 		(at 175.26 52.07 180)
@@
 		)
 		(property "Intersheetrefs" "${INTERSHEET_REFS}"
-			(at 164.1711 52.07 0)
+			(at 163.9897 52.07 0)
 			(effects
 				(font
@@
 		)
 	)
-	(global_label "PWM"
-		(shape input)
-		(at 72.39 72.39 0)
+	(global_label "PWMfilt"
+		(shape output)
+		(at 177.8 27.94 0)
 		(fields_autoplaced yes)
 		(effects
@@
 		)
 		(property "Intersheetrefs" "${INTERSHEET_REFS}"
-			(at 79.548 72.39 0)
+			(at 187.6794 27.94 0)
 			(effects
 				(font
@@
 		)
 	)
-	(global_label "PWMfilt"
-		(shape output)
-		(at 177.8 27.94 0)
+	(global_label "PWMCom"
+		(shape input)
+		(at 236.22 125.73 180)
 		(fields_autoplaced yes)
 		(effects
@@
 				(size 1.27 1.27)
 			)
-			(justify left)
+			(justify right)
 		)
 		(property "Intersheetrefs" "${INTERSHEET_REFS}"
-			(at 187.6794 27.94 0)
+			(at 224.9497 125.73 0)
 			(effects
 				(font
 					(size 1.27 1.27)
 				)
-				(justify left)
+				(justify right)
 				(hide yes)
 			)
@@
 	(symbol
 		(lib_id "power:+5V")
-		(at 71.12 67.31 270)
+		(at 71.12 74.93 270)
 		(unit 1)
 		(exclude_from_sim no)
@@
 		(dnp no)
 		(property "Reference" "#PWR06"
-			(at 67.31 67.31 0)
+			(at 67.31 74.93 0)
 			(effects
 				(font
@@
 		)
 		(property "Value" "+5V"
-			(at 74.93 67.31 90)
+			(at 74.93 74.93 90)
 			(effects
 				(font
@@
 		)
 		(property "Footprint" ""
-			(at 71.12 67.31 0)
+			(at 71.12 74.93 0)
 			(effects
 				(font
@@
 		)
 		(property "Datasheet" ""
-			(at 71.12 67.31 0)
+			(at 71.12 74.93 0)
 			(effects
 				(font
@@
 		)
 		(property "Description" ""
-			(at 71.12 67.31 0)
+			(at 71.12 74.93 0)
 			(effects
 				(font
@@
 	(symbol
 		(lib_id "power:GND")
-		(at 39.37 74.93 270)
-		(unit 1)
-		(exclude_from_sim no)
-		(in_bom yes)
-		(on_board yes)
-		(dnp no)
-		(fields_autoplaced yes)
-		(property "Reference" "#PWR05"
-			(at 33.02 74.93 0)
-			(effects
-				(font
-					(size 1.27 1.27)
-				)
-				(hide yes)
-			)
-		)
-		(property "Value" "GND"
-			(at 35.56 74.93 90)
-			(effects
-				(font
-					(size 1.27 1.27)
-				)
-				(justify right)
-			)
-		)
-		(property "Footprint" ""
-			(at 39.37 74.93 0)
-			(effects
-				(font
-					(size 1.27 1.27)
-				)
-				(hide yes)
-			)
-		)
-		(property "Datasheet" ""
-			(at 39.37 74.93 0)
-			(effects
-				(font
-					(size 1.27 1.27)
-				)
-				(hide yes)
-			)
-		)
-		(property "Description" ""
-			(at 39.37 74.93 0)
-			(effects
-				(font
-					(size 1.27 1.27)
-				)
-				(hide yes)
-			)
-		)
-		(pin "1"
-		)
-		(instances
-			(project "Single_board"
-				(path "/f30854c1-5bc2-470d-aabe-1768a5b01b46"
-					(reference "#PWR05")
-					(unit 1)
-				)
-			)
-		)
-	)
-	(symbol
-		(lib_id "power:GND")
 		(at 29.21 134.62 270)
 		(unit 1)
@@
 	)
 	(sheet
-		(at 43.18 64.77)
-		(size 24.13 13.97)
+		(at 43.18 68.58)
+		(size 24.13 12.7)
 		(fields_autoplaced yes)
 		(stroke
@@
 		)
 		(property "Sheetname" "Keyboard Backlight"
-			(at 43.18 64.0584 0)
+			(at 43.18 67.8684 0)
 			(effects
 				(font
@@
 		)
 		(property "Sheetfile" "backlight.kicad_sch"
-			(at 43.18 79.3246 0)
+			(at 43.18 81.8646 0)
 			(effects
 				(font
@@
 		)
 		(pin "PWR" input
-			(at 67.31 67.31 0)
-			(effects
-				(font
-					(size 1.27 1.27)
-				)
-				(justify right)
-			)
-		)
-		(pin "PWM" input
-			(at 67.31 72.39 0)
+			(at 67.31 74.93 0)
 			(effects
 				(font
@@
 			)
 		)
-		(pin "GND" output
+		(pin "PWMCom" output
 			(at 43.18 74.93 180)
 			(effects
@@
 			(color 255 255 255 1.0000)
 		)
-		(property "Sheetname" "Alarm_lights"
+		(property "Sheetname" "Alarm Lights"
 			(at 240.03 121.2084 0)
 			(effects
@@
 			(effects
 				(font
+					(size 1.27 1.27)
+				)
+				(justify left)
+			)
+		)
+		(pin "PWMCom" output
+			(at 240.03 125.73 180)
+			(effects
+				(font
