File: Boards/Single_board/buttonmatrix.kicad_sch (KiCad schematic)
At the start: 24 parts, among them SW1 +, SW10 5, SW11 2, SW12 9, SW13 PRO, SW14 6, SW15 3, SW16 CLR, SW17 ENTR, SW18 RSET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

Commit message: some progress on the arduino boilerplate
Other:
- title: DSKY Main Board -> DSKY Button Matrix
Changed lines of the file:
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@@
 	(paper "A4")
 	(title_block
-		(title "DSKY Main Board")
+		(title "DSKY Button Matrix")
 		(date "2024-06-02")
 		(rev "0.4.x")

Commit message: fix cherry 3d models in footprints
Parts:
- SW1, SW10, SW11, SW12, SW13, SW14, SW15, SW16, SW17, SW18, SW19, SW2, SW3, SW4, SW5, SW6, SW7, SW8, SW9: footprint Button_Switch_Keyboard:SW_Cherry_MX_1.00u_PCB -> Switch_Misc:SW_Cherry_MX_1.00u_PCB
Changed lines of the file:
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@@
 			)
 		)
-		(property "Footprint" "Button_Switch_Keyboard:SW_Cherry_MX_1.00u_PCB"
+		(property "Footprint" "Switch_Misc:SW_Cherry_MX_1.00u_PCB"
 			(at 140.97 67.31 0)
 			(effects
@@
 			)
 		)
-		(property "Footprint" "Button_Switch_Keyboard:SW_Cherry_MX_1.00u_PCB"
+		(property "Footprint" "Switch_Misc:SW_Cherry_MX_1.00u_PCB"
 			(at 187.96 113.03 0)
 			(effects
@@
 			)
 		)
-		(property "Footprint" "Button_Switch_Keyboard:SW_Cherry_MX_1.00u_PCB"
+		(property "Footprint" "Switch_Misc:SW_Cherry_MX_1.00u_PCB"
 			(at 95.25 67.31 0)
 			(effects
@@
 			)
 		)
-		(property "Footprint" "Button_Switch_Keyboard:SW_Cherry_MX_1.00u_PCB"
+		(property "Footprint" "Switch_Misc:SW_Cherry_MX_1.00u_PCB"
 			(at 118.11 44.45 0)
 			(effects
@@
 			)
 		)
-		(property "Footprint" "Button_Switch_Keyboard:SW_Cherry_MX_1.00u_PCB"
+		(property "Footprint" "Switch_Misc:SW_Cherry_MX_1.00u_PCB"
 			(at 95.25 113.03 0)
 			(effects
@@
 			)
 		)
-		(property "Footprint" "Button_Switch_Keyboard:SW_Cherry_MX_1.00u_PCB"
+		(property "Footprint" "Switch_Misc:SW_Cherry_MX_1.00u_PCB"
 			(at 187.96 67.31 0)
 			(effects
@@
 			)
 		)
-		(property "Footprint" "Button_Switch_Keyboard:SW_Cherry_MX_1.00u_PCB"
+		(property "Footprint" "Switch_Misc:SW_Cherry_MX_1.00u_PCB"
 			(at 95.25 44.45 0)
 			(effects
@@
 			)
 		)
-		(property "Footprint" "Button_Switch_Keyboard:SW_Cherry_MX_1.00u_PCB"
+		(property "Footprint" "Switch_Misc:SW_Cherry_MX_1.00u_PCB"
 			(at 163.83 67.31 0)
 			(effects
@@
 			)
 		)
-		(property "Footprint" "Button_Switch_Keyboard:SW_Cherry_MX_1.00u_PCB"
+		(property "Footprint" "Switch_Misc:SW_Cherry_MX_1.00u_PCB"
 			(at 118.11 67.31 0)
 			(effects
@@
 			)
 		)
-		(property "Footprint" "Button_Switch_Keyboard:SW_Cherry_MX_1.00u_PCB"
+		(property "Footprint" "Switch_Misc:SW_Cherry_MX_1.00u_PCB"
 			(at 140.97 44.45 0)
 			(effects
@@
 			)
 		)
-		(property "Footprint" "Button_Switch_Keyboard:SW_Cherry_MX_1.00u_PCB"
+		(property "Footprint" "Switch_Misc:SW_Cherry_MX_1.00u_PCB"
 			(at 118.11 90.17 0)
 			(effects
@@
 			)
 		)
-		(property "Footprint" "Button_Switch_Keyboard:SW_Cherry_MX_1.00u_PCB"
+		(property "Footprint" "Switch_Misc:SW_Cherry_MX_1.00u_PCB"
 			(at 140.97 113.03 0)
 			(effects
@@
 			)
 		)
-		(property "Footprint" "Button_Switch_Keyboard:SW_Cherry_MX_1.00u_PCB"
+		(property "Footprint" "Switch_Misc:SW_Cherry_MX_1.00u_PCB"
 			(at 163.83 90.17 0)
 			(effects
@@
 			)
 		)
-		(property "Footprint" "Button_Switch_Keyboard:SW_Cherry_MX_1.00u_PCB"
+		(property "Footprint" "Switch_Misc:SW_Cherry_MX_1.00u_PCB"
 			(at 95.25 90.17 0)
 			(effects
@@
 			)
 		)
-		(property "Footprint" "Button_Switch_Keyboard:SW_Cherry_MX_1.00u_PCB"
+		(property "Footprint" "Switch_Misc:SW_Cherry_MX_1.00u_PCB"
 			(at 163.83 113.03 0)
 			(effects
@@
 			)
 		)
-		(property "Footprint" "Button_Switch_Keyboard:SW_Cherry_MX_1.00u_PCB"
+		(property "Footprint" "Switch_Misc:SW_Cherry_MX_1.00u_PCB"
 			(at 163.83 44.45 0)
 			(effects
@@
 			)
 		)
-		(property "Footprint" "Button_Switch_Keyboard:SW_Cherry_MX_1.00u_PCB"
+		(property "Footprint" "Switch_Misc:SW_Cherry_MX_1.00u_PCB"
 			(at 187.96 90.17 0)
 			(effects
@@
 			)
 		)
-		(property "Footprint" "Button_Switch_Keyboard:SW_Cherry_MX_1.00u_PCB"
+		(property "Footprint" "Switch_Misc:SW_Cherry_MX_1.00u_PCB"
 			(at 187.96 44.45 0)
 			(effects
@@
 			)
 		)
-		(property "Footprint" "Button_Switch_Keyboard:SW_Cherry_MX_1.00u_PCB"
+		(property "Footprint" "Switch_Misc:SW_Cherry_MX_1.00u_PCB"
 			(at 118.11 113.03 0)
 			(effects

Commit message: Start RGB LED + hotswap socket redesign of single board
Parts:
- SW1, SW10, SW11, SW12, SW13, SW14, SW15, SW16, SW17, SW18, SW19, SW2, SW3, SW4, SW5, SW6, SW7, SW8, SW9: footprint Switch_Misc:SW_Cherry_MX_1.00u_PCB -> Project Libraries:Kailh_socket_MX
Changed lines of the file:
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@@
 			)
 		)
-		(property "Footprint" "Switch_Misc:SW_Cherry_MX_1.00u_PCB"
+		(property "Footprint" "Project Libraries:Kailh_socket_MX"
 			(at 140.97 67.31 0)
 			(effects
@@
 			)
 		)
-		(property "Footprint" "Switch_Misc:SW_Cherry_MX_1.00u_PCB"
+		(property "Footprint" "Project Libraries:Kailh_socket_MX"
 			(at 187.96 113.03 0)
 			(effects
@@
 			)
 		)
-		(property "Footprint" "Switch_Misc:SW_Cherry_MX_1.00u_PCB"
+		(property "Footprint" "Project Libraries:Kailh_socket_MX"
 			(at 95.25 67.31 0)
 			(effects
@@
 			)
 		)
-		(property "Footprint" "Switch_Misc:SW_Cherry_MX_1.00u_PCB"
+		(property "Footprint" "Project Libraries:Kailh_socket_MX"
 			(at 118.11 44.45 0)
 			(effects
@@
 			)
 		)
-		(property "Footprint" "Switch_Misc:SW_Cherry_MX_1.00u_PCB"
+		(property "Footprint" "Project Libraries:Kailh_socket_MX"
 			(at 95.25 113.03 0)
 			(effects
@@
 			)
 		)
-		(property "Footprint" "Switch_Misc:SW_Cherry_MX_1.00u_PCB"
+		(property "Footprint" "Project Libraries:Kailh_socket_MX"
 			(at 187.96 67.31 0)
 			(effects
@@
 			)
 		)
-		(property "Footprint" "Switch_Misc:SW_Cherry_MX_1.00u_PCB"
+		(property "Footprint" "Project Libraries:Kailh_socket_MX"
 			(at 95.25 44.45 0)
 			(effects
@@
 			)
 		)
-		(property "Footprint" "Switch_Misc:SW_Cherry_MX_1.00u_PCB"
+		(property "Footprint" "Project Libraries:Kailh_socket_MX"
 			(at 163.83 67.31 0)
 			(effects
@@
 			)
 		)
-		(property "Footprint" "Switch_Misc:SW_Cherry_MX_1.00u_PCB"
+		(property "Footprint" "Project Libraries:Kailh_socket_MX"
 			(at 118.11 67.31 0)
 			(effects
@@
 			)
 		)
-		(property "Footprint" "Switch_Misc:SW_Cherry_MX_1.00u_PCB"
+		(property "Footprint" "Project Libraries:Kailh_socket_MX"
 			(at 140.97 44.45 0)
 			(effects
@@
 			)
 		)
-		(property "Footprint" "Switch_Misc:SW_Cherry_MX_1.00u_PCB"
+		(property "Footprint" "Project Libraries:Kailh_socket_MX"
 			(at 118.11 90.17 0)
 			(effects
@@
 			)
 		)
-		(property "Footprint" "Switch_Misc:SW_Cherry_MX_1.00u_PCB"
+		(property "Footprint" "Project Libraries:Kailh_socket_MX"
 			(at 140.97 113.03 0)
 			(effects
@@
 			)
 		)
-		(property "Footprint" "Switch_Misc:SW_Cherry_MX_1.00u_PCB"
+		(property "Footprint" "Project Libraries:Kailh_socket_MX"
 			(at 163.83 90.17 0)
 			(effects
@@
 			)
 		)
-		(property "Footprint" "Switch_Misc:SW_Cherry_MX_1.00u_PCB"
+		(property "Footprint" "Project Libraries:Kailh_socket_MX"
 			(at 95.25 90.17 0)
 			(effects
@@
 			)
 		)
-		(property "Footprint" "Switch_Misc:SW_Cherry_MX_1.00u_PCB"
+		(property "Footprint" "Project Libraries:Kailh_socket_MX"
 			(at 163.83 113.03 0)
 			(effects
@@
 			)
 		)
-		(property "Footprint" "Switch_Misc:SW_Cherry_MX_1.00u_PCB"
+		(property "Footprint" "Project Libraries:Kailh_socket_MX"
 			(at 163.83 44.45 0)
 			(effects
@@
 			)
 		)
-		(property "Footprint" "Switch_Misc:SW_Cherry_MX_1.00u_PCB"
+		(property "Footprint" "Project Libraries:Kailh_socket_MX"
 			(at 187.96 90.17 0)
 			(effects
@@
 			)
 		)
-		(property "Footprint" "Switch_Misc:SW_Cherry_MX_1.00u_PCB"
+		(property "Footprint" "Project Libraries:Kailh_socket_MX"
 			(at 187.96 44.45 0)
 			(effects
@@
 			)
 		)
-		(property "Footprint" "Switch_Misc:SW_Cherry_MX_1.00u_PCB"
+		(property "Footprint" "Project Libraries:Kailh_socket_MX"
 			(at 118.11 113.03 0)
 			(effects

Commit message: Board and 3d models update
Connections:
- net +5V renamed VCC
