File: Boards/Single_board/Single_board.kicad_pcb (KiCad board)
At the start: 2 copper layers, 169.9 x 190.9 mm, 114 parts, among them J1 POWER, J2 ICSP, J3 USB_C_Receptacle_USB2.0_16P, J4 USB_C_Receptacle_USB2.0_16P, J5 USB_C_Receptacle_USB2.0_16P, SW1 +, SW10 5, SW11 2, SW12 9, SW13 PRO, SW14 6, SW15 3, SW16 CLR, SW17 ENTR, SW18 RSET, SW19 KEYREL, SW2 VERB, SW3 NOUN, SW4 0, SW5 7, SW6 -, SW7 4, SW8 1, SW9 8, U2 ATmega328P-A, U3 CH340C

Commit message: Board and 3d models update
Parts:
- added C41: 100nF, Capacitor_SMD:C_0805_2012Metric, B.Cu at (287.5, 208.5)
- added D35: MBR0520LT1G, Diode_SMD:D_SOD-123, B.Cu at (164.9, 132.5)
- D34: value MBR0520LT1G -> SK6812MINI; footprint Diode_SMD:D_SOD-123 -> Project Libraries:SK6812-MINI-E
- moved D34 137.4 mm to (281.7, 208.3), turned to 180 degrees
- moved J2 56.8 mm to (159.0, 108.2), turned to 0 degrees
- moved D32 44.4 mm to (257.0, 220.6)
- moved C39 44.4 mm to (262.9, 220.8)
- moved J3 35.7 mm to (157.3, 92.3), turned to 0 degrees
- moved J1 34.8 mm to (170.6, 109.7)
- moved R45 34.7 mm to (154.0, 90.7)
- moved R44 31.0 mm to (154.0, 94.1), turned to 90 degrees
- moved D33 24.6 mm to (281.7, 183.6)
- moved C40 24.6 mm to (287.5, 183.8)
- moved J4 19.8 mm to (165.0, 92.3), turned to 0 degrees
- moved R3 18.0 mm to (161.6, 90.7)
- moved C38 14.7 mm to (263.5, 206.3)
- moved R2 14.3 mm to (161.6, 94.1), turned to 90 degrees
- moved D31 14.0 mm to (257.0, 206.6)
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Connections:
- D33 pad 1: unconnected-(D33-DOUT-Pad1) -> Net-(D33-DOUT)
- D34 pad 1: 5V1A -> unconnected-(D34-DOUT-Pad1)
- D34 pad 2: Net-(D34-A) -> GND
- J3 pad A4: Net-(D34-A) -> Net-(D35-A)
- J3 pad A9: Net-(D34-A) -> Net-(D35-A)
- J3 pad B4: Net-(D34-A) -> Net-(D35-A)
- J3 pad B9: Net-(D34-A) -> Net-(D35-A)
- R4 pad 1: +5V -> 5V1A
- R5 pad 1: +5V -> 5V1A
- R6 pad 1: +5V -> 5V1A
- R7 pad 1: +5V -> 5V1A
- R8 pad 1: +5V -> 5V1A
Routing:
- added copper zone on F.Cu, net 5V10A
- removed copper zone on F.Cu, net +5V
Other:
- board text added: "Rev. 1.0.0"
- board text removed: "Rev. 0.5.x"

Commit message: Plane layout
Routing:
- net X0: track 0.00 -> 56.2 mm
Changed lines of the file:
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@@
 		)
 		(property "Value" "POWER"
-			(at -4.953 0.2794 0)
+			(at 5.08 0 0)
 			(layer "B.Fab")
 			(effects
@@
 			(pinfunction "Pin_1")
 			(pintype "passive")
+			(thermal_bridge_width 1.5)
 		)
 		(pad "2" thru_hole circle
@@
 			(pinfunction "Pin_2")
 			(pintype "passive")
+			(thermal_bridge_width 1.5)
 		)
 		(model "${KIPRJMOD}/../Libraries/3D/2Pin Terminal Block.step"
@@
 		)
 	)
+	(segment
+		(start 150.8344 163.7538)
+		(end 138.5154 163.7538)
+		(width 0.25)
+		(layer "B.Cu")
+		(net 11)
+	)
+	(segment
+		(start 123.952 178.3172)
+		(end 123.952 198.4664)
+		(width 0.25)
+		(layer "B.Cu")
+		(net 11)
+	)
+	(segment
+		(start 123.952 198.4664)
+		(end 126.1964 200.7108)
+		(width 0.25)
+		(layer "B.Cu")
+		(net 11)
+	)
+	(segment
+		(start 138.5154 163.7538)
+		(end 126.1964 176.0728)
+		(width 0.25)
+		(layer "B.Cu")
+		(net 11)
+	)
+	(segment
+		(start 126.1964 176.0728)
+		(end 123.952 178.3172)
+		(width 0.25)
+		(layer "B.Cu")
+		(net 11)
+	)
 	(zone
 		(net 77)
@@
 		(min_thickness 0.25)
 		(filled_areas_thickness no)
-		(fill
+		(fill yes
 			(thermal_gap 0.5)
 			(thermal_bridge_width 0.5)
@@
 		(min_thickness 0.25)
 		(filled_areas_thickness no)
-		(fill
+		(fill yes
 			(thermal_gap 0.5)
 			(thermal_bridge_width 0.5)

Commit message: Initial autoroute
Routing:
- net Y2: track 0.00 -> 251.1 mm, vias 0 -> 4
- net 5V1A: track 0.00 -> 235.8 mm, vias 0 -> 5
- net X4: track 0.00 -> 229.8 mm, vias 0 -> 2
- net Y1: track 0.00 -> 225.5 mm, vias 0 -> 3
- net Y3: track 0.00 -> 196.5 mm, vias 0 -> 6
- net Net-(D14-DOUT): track 0.00 -> 190.5 mm
- net X3: track 0.00 -> 165.0 mm, vias 0 -> 3
- net 5V10A: track 0.00 -> 133.6 mm, vias 0 -> 68
- net Y0: track 0.00 -> 123.7 mm, vias 0 -> 2
- net X1: track 0.00 -> 112.6 mm, vias 0 -> 4
- net X2: track 0.00 -> 107.4 mm, vias 0 -> 3
- net Net-(U3-UD-): track 0.00 -> 97.3 mm, vias 0 -> 3
- net X0: track 56.2 -> 147.9 mm, vias 0 -> 2
- net Net-(U3-UD+): track 0.00 -> 77.9 mm
- net RESET: track 0.00 -> 73.8 mm
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