File: Boards/Single_board/serial.kicad_sch (KiCad schematic)
At the start: 11 parts, among them J3 USB_C_Receptacle_USB2.0_16P, U3 CH340C

Commit message: Add usb ports and separate power sources. Pending fitting test.
Parts:
- J3: footprint Connector_USB:USB_C_Receptacle_G-Switch_GT-USB-7010ASV -> Project Libraries:USB-C-TH_918-468K2029E50001
Connections:
- net +5V renamed VCC

Commit message: Board and 3d models update
Parts:
- renumbered D34 to D35
Changed lines of the file:
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@@
 		(dnp no)
 		(fields_autoplaced yes)
-		(property "Reference" "D34"
+		(property "Reference" "D35"
 			(at 124.46 41.91 0)
 			(effects
@@
 			(project "Single_board"
 				(path "/f30854c1-5bc2-470d-aabe-1768a5b01b46/2c846281-f7ac-4d2e-99f9-816b435af6ae"
-					(reference "D34")
+					(reference "D35")
 					(unit 1)
 				)

Commit message: Small routing improvements and prepare for JLC order
Parts:
- C1: footprint Capacitor_SMD:C_0805_2012Metric -> Project Libraries:0805 4.7uF
- C2, C3, C4: footprint Capacitor_SMD:C_0805_2012Metric -> Project Libraries:0805 100nF
Changed lines of the file:
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@@
 			)
 		)
-		(property "Footprint" "Capacitor_SMD:C_0805_2012Metric"
+		(property "Footprint" "Project Libraries:0805 4.7uF"
 			(at 166.37 54.61 0)
 			(effects
@@
 			)
 		)
-		(property "Footprint" "Capacitor_SMD:C_0805_2012Metric"
+		(property "Footprint" "Project Libraries:0805 100nF"
 			(at 207.01 52.07 0)
 			(effects
@@
 			)
 		)
-		(property "Footprint" "Capacitor_SMD:C_0805_2012Metric"
+		(property "Footprint" "Project Libraries:0805 100nF"
 			(at 177.8 54.61 0)
 			(effects
@@
 			)
 		)
-		(property "Footprint" "Capacitor_SMD:C_0805_2012Metric"
+		(property "Footprint" "Project Libraries:0805 100nF"
 			(at 220.98 83.82 0)
 			(effects
